File: schematic and pcb/PlayStation 1 Reset Mod.sch (KiCad schematic (older format))
At the start: 17 parts, among them U1 PIC16F18325-ISL

Commit message: updated schematic and PCB
fix issues #1, #2, #3, #5
Parts:
- removed R1: 10k, Resistor_SMD:R_1206_3216Metric_Pad1.42x1.75mm_HandSolder, symbol Device:R
- removed R2: 10k, Resistor_SMD:R_0805_2012Metric_Pad1.15x1.40mm_HandSolder, symbol Device:R
- C1, C2: value CP1_Small -> 0.1uF
Connections:
- wire segments 43 -> 32
Other:
- note added: "PlayStation"
- moved on the sheet: C1, C2
Changed lines of the file:
@@
 EESchema Schematic File Version 4
+LIBS:PlayStation 1 Reset Mod-cache
 EELAYER 29 0
 EELAYER END
@@
 	1    0    0    -1
 $EndComp
-Wire Wire Line
-	5700 3050 5700 3100
-$Comp
-L Device:R R1
-U 1 1 5DA29FC1
-P 5250 3100
-F 0 "R1" V 5350 3100 50  0000 C CNN
-F 1 "10k" V 5250 3100 50  0000 C CNN
-F 2 "Resistor_SMD:R_1206_3216Metric_Pad1.42x1.75mm_HandSolder" V 5180 3100 50  0001 C CNN
-F 3 "~" H 5250 3100 50  0001 C CNN
-	1    5250 3100
-	0    1    1    0
-$EndComp
-Wire Wire Line
-	4850 3100 5000 3100
-Wire Wire Line
-	4850 3100 4850 3450
-Connection ~ 5700 3100
-Wire Wire Line
-	5700 3100 5700 3150
 Text Label 4050 3450 0    50   ~ 0
 VPP\~MCLR
@@
 	3550 3300 3550 3450
 Wire Wire Line
-	5400 3100 5500 3100
-Wire Wire Line
-	4850 3450 5200 3450
-Connection ~ 4850 3450
-Wire Wire Line
-	4000 3450 4850 3450
-Wire Wire Line
 	5200 3550 3850 3550
 Wire Wire Line
@@
 	6200 3650 6900 3650
 Wire Wire Line
-	5050 3750 5050 4600
-Wire Wire Line
-	5050 4600 7050 4600
-Wire Wire Line
-	7050 4600 7050 3400
-$Comp
-L Device:R R2
-U 1 1 5DA62CBE
-P 5250 2950
-F 0 "R2" V 5150 2950 50  0000 C CNN
-F 1 "10k" V 5250 2950 50  0000 C CNN
-F 2 "Resistor_SMD:R_0805_2012Metric_Pad1.15x1.40mm_HandSolder" V 5180 2950 50  0001 C CNN
-F 3 "~" H 5250 2950 50  0001 C CNN
-	1    5250 2950
-	0    1    1    0
-$EndComp
-Wire Wire Line
-	5100 2950 5000 2950
-Wire Wire Line
-	5000 2950 5000 3100
-Connection ~ 5000 3100
-Wire Wire Line
-	5000 3100 5100 3100
-Wire Wire Line
-	5400 2950 5500 2950
-Wire Wire Line
-	5500 2950 5500 3100
-Connection ~ 5500 3100
-Wire Wire Line
-	5500 3100 5700 3100
+	5050 3750 5050 4550
+Wire Wire Line
+	5050 4550 7050 4550
+Wire Wire Line
+	7050 4550 7050 3400
 Wire Wire Line
 	4000 3450 4000 3300
@@
 L Device:CP1_Small C1
 U 1 1 5DA2B48A
-P 6050 2650
-F 0 "C1" H 6141 2650 50  0000 L CNN
-F 1 "CP1_Small" H 6141 2605 50  0001 L CNN
-F 2 "Capacitor_SMD:C_1206_3216Metric_Pad1.42x1.75mm_HandSolder" H 6050 2650 50  0001 C CNN
-F 3 "~" H 6050 2650 50  0001 C CNN
-	1    6050 2650
+P 4900 2800
+F 0 "C1" H 4650 2850 50  0000 L CNN
+F 1 "0.1uF" H 4600 2750 50  0000 L CNN
+F 2 "Capacitor_SMD:C_1206_3216Metric_Pad1.42x1.75mm_HandSolder" H 4900 2800 50  0001 C CNN
+F 3 "~" H 4900 2800 50  0001 C CNN
+	1    4900 2800
 	1    0    0    -1
 $EndComp
@@
 L power:+3.3V #PWR05
 U 1 1 5DA2BBAB
-P 6050 2450
-F 0 "#PWR05" H 6050 2300 50  0001 C CNN
-F 1 "+3.3V" H 6065 2623 50  0000 C CNN
-F 2 "" H 6050 2450 50  0001 C CNN
-F 3 "" H 6050 2450 50  0001 C CNN
-	1    6050 2450
+P 4900 2600
+F 0 "#PWR05" H 4900 2450 50  0001 C CNN
+F 1 "+3.3V" H 4915 2773 50  0000 C CNN
+F 2 "" H 4900 2600 50  0001 C CNN
+F 3 "" H 4900 2600 50  0001 C CNN
+	1    4900 2600
 	1    0    0    -1
 $EndComp
@@
 L power:GND #PWR06
 U 1 1 5DA2C059
-P 6050 2850
-F 0 "#PWR06" H 6050 2600 50  0001 C CNN
-F 1 "GND" H 6055 2677 50  0000 C CNN
-F 2 "" H 6050 2850 50  0001 C CNN
-F 3 "" H 6050 2850 50  0001 C CNN
-	1    6050 2850
-	1    0    0    -1
-$EndComp
-Wire Wire Line
-	6050 2850 6050 2800
-Wire Wire Line
-	6050 2550 6050 2500
+P 4900 3000
+F 0 "#PWR06" H 4900 2750 50  0001 C CNN
+F 1 "GND" H 4905 2827 50  0000 C CNN
+F 2 "" H 4900 3000 50  0001 C CNN
+F 3 "" H 4900 3000 50  0001 C CNN
+	1    4900 3000
+	1    0    0    -1
+$EndComp
+Wire Wire Line
+	4900 3000 4900 2950
+Wire Wire Line
+	4900 2700 4900 2650
 $Comp
 L Device:CP1_Small C2
 U 1 1 5DA61B3C
-P 6350 2650
-F 0 "C2" H 6441 2650 50  0000 L CNN
-F 1 "CP1_Small" H 6441 2605 50  0001 L CNN
-F 2 "Capacitor_SMD:C_0805_2012Metric_Pad1.15x1.40mm_HandSolder" H 6350 2650 50  0001 C CNN
-F 3 "~" H 6350 2650 50  0001 C CNN
-	1    6350 2650
-	1    0    0    -1
-$EndComp
-Wire Wire Line
-	6350 2550 6350 2500
-Wire Wire Line
-	6350 2500 6050 2500
-Connection ~ 6050 2500
-Wire Wire Line
-	6050 2500 6050 2450
-Wire Wire Line
-	6350 2750 6350 2800
-Wire Wire Line
-	6350 2800 6050 2800
-Connection ~ 6050 2800
-Wire Wire Line
-	6050 2800 6050 2750
+P 5200 2800
+F 0 "C2" H 5350 2850 50  0000 L CNN
+F 1 "0.1uF" H 5291 2755 50  0000 L CNN
+F 2 "Capacitor_SMD:C_0805_2012Metric_Pad1.15x1.40mm_HandSolder" H 5200 2800 50  0001 C CNN
+F 3 "~" H 5200 2800 50  0001 C CNN
+	1    5200 2800
+	1    0    0    -1
+$EndComp
+Wire Wire Line
+	5200 2700 5200 2650
+Wire Wire Line
+	5200 2650 4900 2650
+Connection ~ 4900 2650
+Wire Wire Line
+	4900 2650 4900 2600
+Wire Wire Line
+	5200 2900 5200 2950
+Wire Wire Line
+	5200 2950 4900 2950
+Connection ~ 4900 2950
+Wire Wire Line
+	4900 2950 4900 2900
 $Comp
 L Connector:TestPoint TP11
@@
 L power:+3.3V #PWR0101
 U 1 1 5DAB3ABC
-P 7500 3050
-F 0 "#PWR0101" H 7500 2900 50  0001 C CNN
-F 1 "+3.3V" H 7515 3223 50  0000 C CNN
-F 2 "" H 7500 3050 50  0001 C CNN
-F 3 "" H 7500 3050 50  0001 C CNN
-	1    7500 3050
+P 7500 3000
+F 0 "#PWR0101" H 7500 2850 50  0001 C CNN
+F 1 "+3.3V" H 7515 3173 50  0000 C CNN
+F 2 "" H 7500 3000 50  0001 C CNN
+F 3 "" H 7500 3000 50  0001 C CNN
+	1    7500 3000
 	1    0    0    -1
 $EndComp
@@
 L power:GND #PWR0102
 U 1 1 5DAB41BD
-P 7350 3500
-F 0 "#PWR0102" H 7350 3250 50  0001 C CNN
-F 1 "GND" H 7355 3327 50  0000 C CNN
-F 2 "" H 7350 3500 50  0001 C CNN
-F 3 "" H 7350 3500 50  0001 C CNN
-	1    7350 3500
-	1    0    0    -1
-$EndComp
-Wire Wire Line
-	7350 3500 7350 3400
-Wire Wire Line
-	7500 3150 7500 3050
+P 7350 3600
+F 0 "#PWR0102" H 7350 3350 50  0001 C CNN
+F 1 "GND" H 7355 3427 50  0000 C CNN
+F 2 "" H 7350 3600 50  0001 C CNN
+F 3 "" H 7350 3600 50  0001 C CNN
+	1    7350 3600
+	1    0    0    -1
+$EndComp
+Wire Wire Line
+	7350 3600 7350 3400
+Wire Wire Line
+	7500 3150 7500 3000
 Wire Notes Line
 	6500 2750 6500 3850
@@
 Text Label 6300 3950 0    50   ~ 0
 RESET
+Text Notes 6550 2850 0    50   ~ 0
+PlayStation
+Wire Wire Line
+	4000 3450 5200 3450
+Wire Wire Line
+	5700 3050 5700 3150
+Text Label 7350 3550 1    50   ~ 0
+VSS
+Text Label 7500 3150 1    50   ~ 0
+VDD
 $EndSCHEMATC

Commit message: added 0603 capacitor
I've added an extra 0603 capacitor footprint
Parts:
- added C3: 0.1uF, Capacitor_SMD:C_0603_1608Metric_Pad1.05x0.95mm_HandSolder, symbol Device:CP1_Small
Connections:
- wire segments 32 -> 36
Other:
- moved on the sheet: C1, C2
Changed lines of the file:
@@
 L Device:CP1_Small C1
 U 1 1 5DA2B48A
-P 4900 2800
-F 0 "C1" H 4650 2850 50  0000 L CNN
-F 1 "0.1uF" H 4600 2750 50  0000 L CNN
-F 2 "Capacitor_SMD:C_1206_3216Metric_Pad1.42x1.75mm_HandSolder" H 4900 2800 50  0001 C CNN
-F 3 "~" H 4900 2800 50  0001 C CNN
-	1    4900 2800
+P 4950 2400
+F 0 "C1" H 5100 2450 50  0000 L CNN
+F 1 "0.1uF" H 5050 2350 50  0000 L CNN
+F 2 "Capacitor_SMD:C_1206_3216Metric_Pad1.42x1.75mm_HandSolder" H 4950 2400 50  0001 C CNN
+F 3 "~" H 4950 2400 50  0001 C CNN
+	1    4950 2400
 	1    0    0    -1
 $EndComp
@@
 L power:+3.3V #PWR05
 U 1 1 5DA2BBAB
-P 4900 2600
-F 0 "#PWR05" H 4900 2450 50  0001 C CNN
-F 1 "+3.3V" H 4915 2773 50  0000 C CNN
-F 2 "" H 4900 2600 50  0001 C CNN
-F 3 "" H 4900 2600 50  0001 C CNN
-	1    4900 2600
+P 4950 2200
+F 0 "#PWR05" H 4950 2050 50  0001 C CNN
+F 1 "+3.3V" H 4965 2373 50  0000 C CNN
+F 2 "" H 4950 2200 50  0001 C CNN
+F 3 "" H 4950 2200 50  0001 C CNN
+	1    4950 2200
 	1    0    0    -1
 $EndComp
@@
 L power:GND #PWR06
 U 1 1 5DA2C059
-P 4900 3000
-F 0 "#PWR06" H 4900 2750 50  0001 C CNN
-F 1 "GND" H 4905 2827 50  0000 C CNN
-F 2 "" H 4900 3000 50  0001 C CNN
-F 3 "" H 4900 3000 50  0001 C CNN
-	1    4900 3000
+P 4950 2600
+F 0 "#PWR06" H 4950 2350 50  0001 C CNN
+F 1 "GND" H 4955 2427 50  0000 C CNN
+F 2 "" H 4950 2600 50  0001 C CNN
+F 3 "" H 4950 2600 50  0001 C CNN
+	1    4950 2600
 	1    0    0    -1
 $EndComp
 Wire Wire Line
-	4900 3000 4900 2950
+	4950 2600 4950 2550
 Wire Wire Line
-	4900 2700 4900 2650
+	4950 2300 4950 2250
 $Comp
 L Device:CP1_Small C2
 U 1 1 5DA61B3C
-P 5200 2800
-F 0 "C2" H 5350 2850 50  0000 L CNN
-F 1 "0.1uF" H 5291 2755 50  0000 L CNN
-F 2 "Capacitor_SMD:C_0805_2012Metric_Pad1.15x1.40mm_HandSolder" H 5200 2800 50  0001 C CNN
-F 3 "~" H 5200 2800 50  0001 C CNN
-	1    5200 2800
+P 5400 2400
+F 0 "C2" H 5550 2450 50  0000 L CNN
+F 1 "0.1uF" H 5491 2355 50  0000 L CNN
+F 2 "Capacitor_SMD:C_0805_2012Metric_Pad1.15x1.40mm_HandSolder" H 5400 2400 50  0001 C CNN
+F 3 "~" H 5400 2400 50  0001 C CNN
+	1    5400 2400
 	1    0    0    -1
 $EndComp
 Wire Wire Line
-	5200 2700 5200 2650
+	5400 2300 5400 2250
 Wire Wire Line
-	5200 2650 4900 2650
-Connection ~ 4900 2650
+	5400 2250 4950 2250
+Connection ~ 4950 2250
 Wire Wire Line
-	4900 2650 4900 2600
+	4950 2250 4950 2200
 Wire Wire Line
-	5200 2900 5200 2950
+	5400 2500 5400 2550
 Wire Wire Line
-	5200 2950 4900 2950
-Connection ~ 4900 2950
+	5400 2550 4950 2550
+Connection ~ 4950 2550
 Wire Wire Line
-	4900 2950 4900 2900
+	4950 2550 4950 2500
 $Comp
 L Connector:TestPoint TP11
@@
 Text Label 7500 3150 1    50   ~ 0
 VDD
+$Comp
+L Device:CP1_Small C3
+U 1 1 5DABA497
+P 5800 2400
+F 0 "C3" H 5950 2450 50  0000 L CNN
+F 1 "0.1uF" H 5891 2355 50  0000 L CNN
+F 2 "Capacitor_SMD:C_0603_1608Metric_Pad1.05x0.95mm_HandSolder" H 5800 2400 50  0001 C CNN
+F 3 "~" H 5800 2400 50  0001 C CNN
+	1    5800 2400
+	1    0    0    -1
+$EndComp
+Wire Wire Line
+	5800 2300 5800 2250
+Wire Wire Line
+	5800 2250 5400 2250
+Connection ~ 5400 2250
+Wire Wire Line
+	5800 2500 5800 2550
+Wire Wire Line
+	5800 2550 5400 2550
+Connection ~ 5400 2550
 $EndSCHEMATC

Commit message: minor addition to schematic
added rectangle around the 3 caps on the schematic with text indicating to only install one
Other:
- note added: "* Only install one cap"
- moved on the sheet: C1, C2, C3
Changed lines of the file:
@@
 L Device:CP1_Small C1
 U 1 1 5DA2B48A
-P 4950 2400
-F 0 "C1" H 5100 2450 50  0000 L CNN
-F 1 "0.1uF" H 5050 2350 50  0000 L CNN
-F 2 "Capacitor_SMD:C_1206_3216Metric_Pad1.42x1.75mm_HandSolder" H 4950 2400 50  0001 C CNN
-F 3 "~" H 4950 2400 50  0001 C CNN
-	1    4950 2400
+P 4800 2250
+F 0 "C1" H 4950 2300 50  0000 L CNN
+F 1 "0.1uF" H 4900 2200 50  0000 L CNN
+F 2 "Capacitor_SMD:C_1206_3216Metric_Pad1.42x1.75mm_HandSolder" H 4800 2250 50  0001 C CNN
+F 3 "~" H 4800 2250 50  0001 C CNN
+	1    4800 2250
 	1    0    0    -1
 $EndComp
@@
 L power:+3.3V #PWR05
 U 1 1 5DA2BBAB
-P 4950 2200
-F 0 "#PWR05" H 4950 2050 50  0001 C CNN
-F 1 "+3.3V" H 4965 2373 50  0000 C CNN
-F 2 "" H 4950 2200 50  0001 C CNN
-F 3 "" H 4950 2200 50  0001 C CNN
-	1    4950 2200
+P 4800 2050
+F 0 "#PWR05" H 4800 1900 50  0001 C CNN
+F 1 "+3.3V" H 4815 2223 50  0000 C CNN
+F 2 "" H 4800 2050 50  0001 C CNN
+F 3 "" H 4800 2050 50  0001 C CNN
+	1    4800 2050
 	1    0    0    -1
 $EndComp
@@
 L power:GND #PWR06
 U 1 1 5DA2C059
-P 4950 2600
-F 0 "#PWR06" H 4950 2350 50  0001 C CNN
-F 1 "GND" H 4955 2427 50  0000 C CNN
-F 2 "" H 4950 2600 50  0001 C CNN
-F 3 "" H 4950 2600 50  0001 C CNN
-	1    4950 2600
+P 4800 2450
+F 0 "#PWR06" H 4800 2200 50  0001 C CNN
+F 1 "GND" H 4805 2277 50  0000 C CNN
+F 2 "" H 4800 2450 50  0001 C CNN
+F 3 "" H 4800 2450 50  0001 C CNN
+	1    4800 2450
 	1    0    0    -1
 $EndComp
 Wire Wire Line
-	4950 2600 4950 2550
+	4800 2450 4800 2400
 Wire Wire Line
-	4950 2300 4950 2250
+	4800 2150 4800 2100
 $Comp
 L Device:CP1_Small C2
 U 1 1 5DA61B3C
-P 5400 2400
-F 0 "C2" H 5550 2450 50  0000 L CNN
-F 1 "0.1uF" H 5491 2355 50  0000 L CNN
-F 2 "Capacitor_SMD:C_0805_2012Metric_Pad1.15x1.40mm_HandSolder" H 5400 2400 50  0001 C CNN
-F 3 "~" H 5400 2400 50  0001 C CNN
-	1    5400 2400
+P 5250 2250
+F 0 "C2" H 5400 2300 50  0000 L CNN
+F 1 "0.1uF" H 5341 2205 50  0000 L CNN
+F 2 "Capacitor_SMD:C_0805_2012Metric_Pad1.15x1.40mm_HandSolder" H 5250 2250 50  0001 C CNN
+F 3 "~" H 5250 2250 50  0001 C CNN
+	1    5250 2250
 	1    0    0    -1
 $EndComp
 Wire Wire Line
-	5400 2300 5400 2250
+	5250 2150 5250 2100
 Wire Wire Line
-	5400 2250 4950 2250
-Connection ~ 4950 2250
+	5250 2100 4800 2100
+Connection ~ 4800 2100
 Wire Wire Line
-	4950 2250 4950 2200
+	4800 2100 4800 2050
 Wire Wire Line
-	5400 2500 5400 2550
+	5250 2350 5250 2400
 Wire Wire Line
-	5400 2550 4950 2550
-Connection ~ 4950 2550
+	5250 2400 4800 2400
+Connection ~ 4800 2400
 Wire Wire Line
-	4950 2550 4950 2500
+	4800 2400 4800 2350
 $Comp
 L Connector:TestPoint TP11
@@
 L Device:CP1_Small C3
 U 1 1 5DABA497
-P 5800 2400
-F 0 "C3" H 5950 2450 50  0000 L CNN
-F 1 "0.1uF" H 5891 2355 50  0000 L CNN
-F 2 "Capacitor_SMD:C_0603_1608Metric_Pad1.05x0.95mm_HandSolder" H 5800 2400 50  0001 C CNN
-F 3 "~" H 5800 2400 50  0001 C CNN
-	1    5800 2400
+P 5650 2250
+F 0 "C3" H 5800 2300 50  0000 L CNN
+F 1 "0.1uF" H 5741 2205 50  0000 L CNN
+F 2 "Capacitor_SMD:C_0603_1608Metric_Pad1.05x0.95mm_HandSolder" H 5650 2250 50  0001 C CNN
+F 3 "~" H 5650 2250 50  0001 C CNN
+	1    5650 2250
 	1    0    0    -1
 $EndComp
 Wire Wire Line
-	5800 2300 5800 2250
+	5650 2150 5650 2100
 Wire Wire Line
-	5800 2250 5400 2250
-Connection ~ 5400 2250
+	5650 2100 5250 2100
+Connection ~ 5250 2100
 Wire Wire Line
-	5800 2500 5800 2550
+	5650 2350 5650 2400
 Wire Wire Line
-	5800 2550 5400 2550
-Connection ~ 5400 2550
+	5650 2400 5250 2400
+Connection ~ 5250 2400
+Wire Notes Line
+	4650 1800 4650 2700
+Wire Notes Line
+	4650 2700 6000 2700
+Wire Notes Line
+	6000 2700 6000 1800
+Wire Notes Line
+	6000 1800 4650 1800
+Text Notes 5100 1900 0    50   ~ 0
+* Only install one cap
 $EndSCHEMATC

Commit message: general update
Parts:
- C1, C2, C3: symbol Device:CP1_Small -> Device:C_Polarized_Small_US
Changed lines of the file:
@@
 EESchema Schematic File Version 4
-LIBS:PlayStation 1 Reset Mod-cache
-EELAYER 29 0
+EELAYER 30 0
 EELAYER END
 $Descr A4 11693 8268
@@
 $EndComp
 $Comp
-L Device:CP1_Small C1
-U 1 1 5DA2B48A
-P 4800 2250
-F 0 "C1" H 4950 2300 50  0000 L CNN
-F 1 "0.1uF" H 4900 2200 50  0000 L CNN
-F 2 "Capacitor_SMD:C_1206_3216Metric_Pad1.42x1.75mm_HandSolder" H 4800 2250 50  0001 C CNN
-F 3 "~" H 4800 2250 50  0001 C CNN
-	1    4800 2250
-	1    0    0    -1
-$EndComp
-$Comp
 L power:+3.3V #PWR05
 U 1 1 5DA2BBAB
@@
 	4800 2150 4800 2100
 $Comp
-L Device:CP1_Small C2
+L Device:C_Polarized_Small_US C2
 U 1 1 5DA61B3C
 P 5250 2250
@@
 VDD
 $Comp
-L Device:CP1_Small C3
+L Device:C_Polarized_Small_US C3
 U 1 1 5DABA497
 P 5650 2250
@@
 Text Notes 5100 1900 0    50   ~ 0
 * Only install one cap
+$Comp
+L Device:C_Polarized_Small_US C1
+U 1 1 5DA2B48A
+P 4800 2250
+F 0 "C1" H 4950 2300 50  0000 L CNN
+F 1 "0.1uF" H 4900 2200 50  0000 L CNN
+F 2 "Capacitor_SMD:C_1206_3216Metric_Pad1.42x1.75mm_HandSolder" H 4800 2250 50  0001 C CNN
+F 3 "~" H 4800 2250 50  0001 C CNN
+	1    4800 2250
+	1    0    0    -1
+$EndComp
 $EndSCHEMATC
